File: kicad/Atari_Input.kicad_sch (KiCad schematic)
At the start: 12 parts

Commit message: a
Parts:
- removed U?: ATmega32U2-M, Package_DFN_QFN:QFN-32-1EP_5x5mm_P0.5mm_EP3.1x3.1mm, symbol MCU_Microchip_ATmega:ATmega32U2-M
- added U?: AT90USB82-16M, Package_DFN_QFN:QFN-32-1EP_5x5mm_P0.5mm_EP3.6x3.6mm, symbol MCU_Microchip_AVR:AT90USB82-16M
Connections:
- net GND: now also U?.28 (UGND), U?.3 (GND), U?.33 (GND)
- net VCC: now also U?.31 (UVCC)
- net ~RESET: now also U?.24 (PC1/~RESET)
- net at C?.2, Y?.4: now also U?.1 (XTAL1)
- net at C?.2, Y?.1: now also U?.2 (PC0/XTAL2)
- net at C?.2: now also U?.27 (UCAP)
- net at J?.3 (D+): now also U?.29 (D+)
- net at J?.2 (D-): now also U?.30 (D-)
- new net: U?.32 (AVCC), U?.4 (VCC)
Changed lines of the file:
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@@
-(kicad_sch (version 20210126) (generator eeschema)
+(kicad_sch (version 20210406) (generator eeschema)
   (paper "A4")
   (junction (at 20.32 63.5) (diameter 0.9144) (color 0 0 0 0))
@@
   (junction (at 50.8 48.26) (diameter 0.9144) (color 0 0 0 0))
   (junction (at 77.47 22.86) (diameter 0.9144) (color 0 0 0 0))
-  (junction (at 77.47 30.48) (diameter 0.9144) (color 0 0 0 0))
   (junction (at 77.47 101.6) (diameter 0.9144) (color 0 0 0 0))
-  (junction (at 80.01 30.48) (diameter 0.9144) (color 0 0 0 0))
   (junction (at 127 96.52) (diameter 0.9144) (color 0 0 0 0))
   (junction (at 128.27 29.21) (diameter 0.9144) (color 0 0 0 0))
@@
     (stroke (width 0) (type solid) (color 0 0 0 0))
   )
-  (wire (pts (xy 77.47 30.48) (xy 80.01 30.48))
-    (stroke (width 0) (type solid) (color 0 0 0 0))
-  )
   (wire (pts (xy 77.47 101.6) (xy 77.47 110.49))
     (stroke (width 0) (type solid) (color 0 0 0 0))
@@
     (pin "6")
   )
-  (symbol (lib_id "MCU_Microchip_ATmega:ATmega32U2-M") (at 80.01 66.04 0) (unit 1)
-    (in_bom yes) (on_board yes)
+  (symbol (lib_id "MCU_Microchip_AVR:AT90USB82-16M") (at 80.01 66.04 0) (unit 1)
+    (in_bom yes) (on_board yes) (fields_autoplaced)
     (property "Reference" "U?" (id 0) (at 80.01 104.14 0))
-    (property "Value" "ATmega32U2-M" (id 1) (at 80.01 106.68 0))
-    (property "Footprint" "Package_DFN_QFN:QFN-32-1EP_5x5mm_P0.5mm_EP3.1x3.1mm" (id 2) (at 80.01 66.04 0)
+    (property "Value" "AT90USB82-16M" (id 1) (at 80.01 106.68 0))
+    (property "Footprint" "Package_DFN_QFN:QFN-32-1EP_5x5mm_P0.5mm_EP3.6x3.6mm" (id 2) (at 80.01 66.04 0)
       (effects (font (size 1.27 1.27) italic) hide)
     )
-    (property "Datasheet" "http://ww1.microchip.com/downloads/en/DeviceDoc/doc7799.pdf" (id 3) (at 80.01 66.04 0)
+    (property "Datasheet" "http://ww1.microchip.com/downloads/en/DeviceDoc/doc7707.pdf" (id 3) (at 80.01 66.04 0)
       (effects (font (size 1.27 1.27)) hide)
     )
@@
       (reference "R?") (unit 1) (value "10k") (footprint "")
     )
-    (path "/39354c90-a6dc-46bb-a7ec-470154c01035"
-      (reference "U?") (unit 1) (value "ATmega32U2-M") (footprint "Package_DFN_QFN:QFN-32-1EP_5x5mm_P0.5mm_EP3.1x3.1mm")
+    (path "/757e971f-2ef8-45ab-a407-6db14e2038df"
+      (reference "U?") (unit 1) (value "AT90USB82-16M") (footprint "Package_DFN_QFN:QFN-32-1EP_5x5mm_P0.5mm_EP3.6x3.6mm")
     )
     (path "/857a82dc-59c9-4879-9554-ed6d5f066120"

Commit message: a
Parts:
- removed C?: 1uF, symbol Device:C
- removed J?: Keyboard, symbol Connector:Mini-DIN-6
- removed J?: Mouse, symbol Connector:Mini-DIN-6
- removed J?: USB_B, symbol Connector:USB_B
- removed R?: 10k, symbol Device:R
- removed U?: AT90USB82-16M, Package_DFN_QFN:QFN-32-1EP_5x5mm_P0.5mm_EP3.6x3.6mm, symbol MCU_Microchip_AVR:AT90USB82-16M
- added J?: SETUP, symbol Connector:USB_B
- added J?: AVR-ISP-6, Connector_IDC:IDC-Header_2x03_P2.54mm_Vertical, symbol Connector:AVR-ISP-6
- added J?: DONGLE, Connector_USB:USB_A_Molex_67643_Horizontal, symbol Connector:USB_A
- added R?: 10k, symbol Device:R
- added U?: ATmega328P-MM, Package_DFN_QFN:QFN-28-1EP_4x4mm_P0.45mm_EP2.4x2.4mm, symbol MCU_Microchip_ATmega:ATmega328P-MM
Connections:
- net GND: now also J?.4 (GND), J?.4 (GND), J?.5 (Shield), J?.5 (Shield), J?.6 (GND), U?.18 (GND), U?.29 (GND), U?.4 (GND)
- net VCC: now also J?.1 (VBUS), J?.1 (VBUS), J?.2 (VCC), R?.2, U?.16 (AVCC), U?.17 (AREF), U?.3 (VCC)
- net ~RESET: now also J?.5 (~RST), R?.1, U?.25 (~RESET~/PC6)
- net at C?.2, Y?.4: now also U?.5 (XTAL1/PB6)
- net at C?.2, Y?.1: now also U?.6 (XTAL2/PB7)
- no-connect marks 4 -> 0
Other:
- moved on the sheet: C?, J?, Y?
